Commit message: change usv plugin param

File: catkin_ws/src/marine_duckiebot/marine_duckiebot_description/urdf/mybot.xacro (robot description, xacro)
@@ -151,10 +151,10 @@
     <inertial>
       <mass value="6.65" />
-      <origin xyz="0 0 0" rpy="0 0 0"/>
+      <origin xyz="1.135 0 0" rpy="0 0 0"/>
       <box_inertia m="${cameraMass}" x="${cameraSize}" y="${cameraSize}" z="${cameraSize}" />
       <inertia ixx="0.0001" ixy="0" ixz="0" iyy="0.0001" iyz="0" izz="0.0001" />
     </inertial>
   </link>
-  <joint name="weight_joint" type="continuous">
+  <joint name="weight_joint" type="fixed">
     <axis xyz="0 0 0" />
     <origin xyz="-0.2 0 0.0" rpy="0 0.0 0"/>

File: catkin_ws/src/marine_duckiebot/marine_duckiebot_description/urdf/plugin/usv_gazebo_dynamics_plugin_duckiebot.xacro (robot description, xacro)
@@ -2,15 +2,18 @@
 <robot xmlns:xacro="http://ros.org/wiki/xacro">
   <xacro:macro name="usv_gazebo" params="name">
-    <!--Gazebo Plugin for simulating Duckiebot dynamics-->
+    <!--Gazebo Plugin for simulating
+    Duckiebot dynamics-->
     <gazebo >
       <!--<plugin name="heron_dynamic" filename="libheron_gazebo_plugins.so">-->
-      <plugin name="usv_dynamics_${name}" filename="libusv_gazebo_dynamics_plugin.so">
+      <plugin name="usv_dynamics_${name}"
+       filename="
+       libusv_gazebo_dynamics_plugin.so">
 	<bodyName>base_footprint</bodyName>
 	<waterLevel>0</waterLevel>
 	<waterDensity>997.8</waterDensity>
 	<cmdTimeout>1.0</cmdTimeout>
-	<xDotU>5</xDotU>
-	<yDotV>5</yDotV>
-	<nDotR>0.5</nDotR>
+	<xDotU>5.0</xDotU>
+	<yDotV>5.0</yDotV>
+	<nDotR>1.0</nDotR>
 	<xU>20.0</xU>
 	<xUU>0.0</xUU>
@@ -23,6 +26,6 @@
 	<nRR>0.0</nRR>
 	<maxCmd>1.0</maxCmd>
-	<maxForceFwd>70</maxForceFwd>
-	<maxForceRev>-70</maxForceRev>
+	<maxForceFwd>60</maxForceFwd>
+	<maxForceRev>-60</maxForceRev>
 	<boatArea>0.24</boatArea>
 	<boatWidth>0.6</boatWidth>

File: catkin_ws/src/marine_duckiebot/marine_duckiebot_description/urdf/wheel.urdf.xacro (robot description, xacro)
@@ -69,5 +69,5 @@
 			</actuator>
 			<joint name="${wheel_prefix}_wheel_hinge">
-				<hardwareInterface>VelocityJointInterface</hardwareInterface>
+				<hardwareInterface>hardware_interface/VelocityJointInterface</hardwareInterface>
 			</joint>
 		</transmission>
