Commit message: change for lab 1

File: catkin_ws/src/robotx_forum_tutorials/kingfisher_gazebo/urdf/base_gazebo.xacro (robot description, xacro)
@@ -33,3 +33,7 @@
   </xacro:if>
   <xacro:kingfisher_gazebo_camera name="kingfisher"/>
+  <xacro:include filename="$(find velodyne_description)/urdf/VLP-16.urdf.xacro"/>
+  <VLP-16 parent="base_link" name="velodyne" topic="/velodyne_points" hz="10" samples="440">
+    <origin xyz="0 0 0.17" rpy="0 0 0" />
+  </VLP-16>
 </robot>

File: catkin_ws/src/robotx_forum_tutorials/usv_gazebo_plugins/urdf/usv_gazebo_dynamics_plugin.xacro (robot description, xacro)
@@ -7,5 +7,5 @@
       <plugin name="usv_dynamics_${name}" filename="libusv_gazebo_dynamics_plugin.so">
 	<bodyName>base_footprint</bodyName>
-	<waterLevel>5.0</waterLevel>
+	<waterLevel>0.0</waterLevel>
 	<waterDensity>997.8</waterDensity>
 	<cmdTimeout>1.0</cmdTimeout>
